File: OpenAmiga600FastRamExpansion.kicad_pcb (KiCad board)
At the start: 2 copper layers, 72.3 x 72.5 mm, 27 parts, among them J1 MC68000_PLCC68, P1 JTAG_CONNECTOR, P98 SCREW_HOLE, P99 OSHW_LOGO, U1 74LS157, U2 74LS157, U3 HYB5118160BSJ, U4 HYB5118160BSJ, U5 ATF1502AS-10JU44

Commit message: More stitching
Routing:
- net GND: vias 146 -> 160
Changed lines of the file:
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@@
     (thickness 1.6)
     (drawings 102)
-    (tracks 1199)
+    (tracks 1213)
     (zones 0)
     (modules 27)
@@
     (tags "capacitor handsolder")
     (attr smd)
-    (fp_text reference C1 (at 3.05 0 270) (layer F.SilkS)
+    (fp_text reference C1 (at 3.164 0 270) (layer F.SilkS)
       (effects (font (size 1 1) (thickness 0.15)))
     )
@@
   (via (at 125.76175 88.392) (size 0.6) (drill 0.4) (layers F.Cu B.Cu) (net 18))
   (via (at 122.809 88.392) (size 0.6) (drill 0.4) (layers F.Cu B.Cu) (net 18))
-  (via (at 132.9055 88.392) (size 0.6) (drill 0.4) (layers F.Cu B.Cu) (net 18))
+  (via (at 133.4135 88.392) (size 0.6) (drill 0.4) (layers F.Cu B.Cu) (net 18))
   (via (at 112.268 117.856) (size 0.6) (drill 0.4) (layers F.Cu B.Cu) (net 18))
   (via (at 112.268 110.49) (size 0.6) (drill 0.4) (layers F.Cu B.Cu) (net 18))
@@
   (via (at 173.355 97.028) (size 0.6) (drill 0.4) (layers F.Cu B.Cu) (net 18))
   (via (at 176.3395 96.4565) (size 0.6) (drill 0.4) (layers F.Cu B.Cu) (net 18))
-  (via (at 165.608 79.6925) (size 0.6) (drill 0.4) (layers F.Cu B.Cu) (net 18))
+  (via (at 165.608 79.502) (size 0.6) (drill 0.4) (layers F.Cu B.Cu) (net 18))
+  (via (at 166.116 93.726) (size 0.6) (drill 0.4) (layers F.Cu B.Cu) (net 18))
+  (via (at 166.878 87.503) (size 0.6) (drill 0.4) (layers F.Cu B.Cu) (net 18))
+  (via (at 153.416 82.042) (size 0.6) (drill 0.4) (layers F.Cu B.Cu) (net 18))
+  (via (at 156.21 82.042) (size 0.6) (drill 0.4) (layers F.Cu B.Cu) (net 18))
+  (via (at 152.7175 76.708) (size 0.6) (drill 0.4) (layers F.Cu B.Cu) (net 18))
+  (via (at 135.89 78.867) (size 0.6) (drill 0.4) (layers F.Cu B.Cu) (net 18))
+  (via (at 132.0546 78.867) (size 0.6) (drill 0.4) (layers F.Cu B.Cu) (net 18))
+  (via (at 130.7465 78.867) (size 0.6) (drill 0.4) (layers F.Cu B.Cu) (net 18))
+  (via (at 129.4765 78.867) (size 0.6) (drill 0.4) (layers F.Cu B.Cu) (net 18))
+  (via (at 126.3015 61.976) (size 0.6) (drill 0.4) (layers F.Cu B.Cu) (net 18))
+  (via (at 123.7615 122.1105) (size 0.6) (drill 0.4) (layers F.Cu B.Cu) (net 18))
+  (via (at 141.859 106.426) (size 0.6) (drill 0.4) (layers F.Cu B.Cu) (net 18))
+  (via (at 144.145 107.696) (size 0.6) (drill 0.4) (layers F.Cu B.Cu) (net 18))
+  (via (at 144.145 110.236) (size 0.6) (drill 0.4) (layers F.Cu B.Cu) (net 18))
   (segment (start 165.6 76.075) (end 167.925 76.075) (width 0.5) (layer F.Cu) (net 19))
   (segment (start 168.255 75.745) (end 168.255 74.36) (width 0.5) (layer F.Cu) (net 19))

Commit message: More and more stitching
Routing:
- net GND: vias 160 -> 162
Changed lines of the file:
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@@
     (thickness 1.6)
     (drawings 102)
-    (tracks 1213)
+    (tracks 1215)
     (zones 0)
     (modules 27)
@@
   (via (at 144.145 107.696) (size 0.6) (drill 0.4) (layers F.Cu B.Cu) (net 18))
   (via (at 144.145 110.236) (size 0.6) (drill 0.4) (layers F.Cu B.Cu) (net 18))
+  (via (at 147.32 91.2495) (size 0.6) (drill 0.4) (layers F.Cu B.Cu) (net 18))
+  (via (at 147.4216 93.6244) (size 0.6) (drill 0.4) (layers F.Cu B.Cu) (net 18))
   (segment (start 165.6 76.075) (end 167.925 76.075) (width 0.5) (layer F.Cu) (net 19))
   (segment (start 168.255 75.745) (end 168.255 74.36) (width 0.5) (layer F.Cu) (net 19))

Commit message: More and more and more stitching
Routing:
- net GND: vias 162 -> 168
Changed lines of the file:
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@@
     (thickness 1.6)
     (drawings 102)
-    (tracks 1215)
+    (tracks 1221)
     (zones 0)
     (modules 27)
@@
   (via (at 147.32 91.2495) (size 0.6) (drill 0.4) (layers F.Cu B.Cu) (net 18))
   (via (at 147.4216 93.6244) (size 0.6) (drill 0.4) (layers F.Cu B.Cu) (net 18))
+  (via (at 144.526 91.44) (size 0.6) (drill 0.4) (layers F.Cu B.Cu) (net 18))
+  (via (at 142.748 91.44) (size 0.6) (drill 0.4) (layers F.Cu B.Cu) (net 18))
+  (via (at 144.78 93.6244) (size 0.6) (drill 0.4) (layers F.Cu B.Cu) (net 18))
+  (via (at 145.9865 93.6244) (size 0.5) (drill 0.4) (layers F.Cu B.Cu) (net 18))
+  (via (at 142.0114 82.042) (size 0.6) (drill 0.4) (layers F.Cu B.Cu) (net 18))
+  (via (at 143.51 78.867) (size 0.6) (drill 0.4) (layers F.Cu B.Cu) (net 18))
   (segment (start 165.6 76.075) (end 167.925 76.075) (width 0.5) (layer F.Cu) (net 19))
   (segment (start 168.255 75.745) (end 168.255 74.36) (width 0.5) (layer F.Cu) (net 19))
