File: OpenAmiga600FastRamExpansion.kicad_pcb (KiCad board)
At the start: 2 copper layers, 72.3 x 72.5 mm, 27 parts, among them J1 MC68000_PLCC68, P1 JTAG_CONNECTOR, P98 SCREW_HOLE, P99 OSHW_LOGO, U1 74LS157, U2 74LS157, U3 HYB5118160BSJ, U4 HYB5118160BSJ, U5 ATF1502AS-10JU44

Commit message: Add JTAG pinout
Other:
- board text added: "1"
- board text added: "1. TCK 2. GND 3. TDO 4. VCC"
- board text added: "10"
- board text added: "2"
- board text added: "3"
- board text added: "4"
- board text added: "5"
- board text added: "5. TMS 9. TDI 10. GND"
- board text added: "6"
- board text added: "7"
- board text added: "8"
- board text added: "9"
- board text added: "JTAG PINOUT"
Changed lines of the file:
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@@
   (general
     (thickness 1.6)
-    (drawings 103)
+    (drawings 128)
     (tracks 1225)
     (zones 0)
@@
     (tags "capacitor handsolder")
     (attr smd)
-    (fp_text reference C4 (at 3.048 0 270) (layer B.SilkS)
+    (fp_text reference C4 (at -3.1035 0 270) (layer B.SilkS)
       (effects (font (size 1 1) (thickness 0.15)) (justify mirror))
     )
@@
     (pad 1 thru_hole circle (at 1.325825 -1.325825) (size 0.8 0.8) (drill 0.5) (layers *.Cu *.Mask)
       (net 18 GND) (zone_connect 2))
+  )
+  (gr_arc (start 126.24 68.0165) (end 126.24 67.5085) (angle -90) (layer B.SilkS) (width 0.2))
+  (gr_arc (start 126.24 77.9225) (end 125.732 77.9225) (angle -90) (layer B.SilkS) (width 0.2))
+  (gr_arc (start 151.3225 77.9225) (end 151.3225 78.4305) (angle -90) (layer B.SilkS) (width 0.2))
+  (gr_arc (start 151.3225 68.0165) (end 151.8305 68.0165) (angle -90) (layer B.SilkS) (width 0.2))
+  (gr_line (start 126.24 67.5085) (end 151.3225 67.5085) (layer B.SilkS) (width 0.2))
+  (gr_line (start 125.732 77.9225) (end 125.732 68.0165) (layer B.SilkS) (width 0.2))
+  (gr_line (start 151.3225 78.4305) (end 126.24 78.4305) (layer B.SilkS) (width 0.2))
+  (gr_line (start 151.8305 68.0165) (end 151.8305 77.9225) (layer B.SilkS) (width 0.2))
+  (gr_text "5. TMS\n9. TDI\n10. GND" (at 132.6535 72.144) (layer B.SilkS)
+    (effects (font (size 1 1) (thickness 0.2)) (justify left mirror))
+  )
+  (gr_text "1. TCK\n2. GND\n3. TDO\n4. VCC" (at 138.813 72.994) (layer B.SilkS)
+    (effects (font (size 1 1) (thickness 0.2)) (justify left mirror))
+  )
+  (gr_text "JTAG\nPINOUT" (at 145.2265 70.5565) (layer B.SilkS)
+    (effects (font (size 1.5 1.5) (thickness 0.3)) (justify mirror))
+  )
+  (gr_line (start 140.083 73.593498) (end 140.083 77.530498) (layer B.SilkS) (width 0.2))
+  (gr_line (start 150.243 73.593498) (end 140.083 73.593498) (layer B.SilkS) (width 0.2))
+  (gr_line (start 150.243 77.530498) (end 150.243 73.593498) (layer B.SilkS) (width 0.2))
+  (gr_line (start 140.083 77.530498) (end 150.243 77.530498) (layer B.SilkS) (width 0.2))
+  (gr_text 9 (at 148.592 74.609498) (layer B.SilkS)
+    (effects (font (size 1 1) (thickness 0.2)) (justify mirror))
+  )
+  (gr_text 10 (at 148.592 76.387498) (layer B.SilkS)
+    (effects (font (size 1 1) (thickness 0.2)) (justify mirror))
+  )
+  (gr_text 7 (at 146.71875 74.609498) (layer B.SilkS)
+    (effects (font (size 1 1) (thickness 0.2)) (justify mirror))
+  )
+  (gr_text 5 (at 145.0995 74.609498) (layer B.SilkS)
+    (effects (font (size 1 1) (thickness 0.2)) (justify mirror))
+  )
+  (gr_text 8 (at 146.71875 76.387498) (layer B.SilkS)
+    (effects (font (size 1 1) (thickness 0.2)) (justify mirror))
+  )
+  (gr_text 6 (at 145.0995 76.387498) (layer B.SilkS)
+    (effects (font (size 1 1) (thickness 0.2)) (justify mirror))
+  )
+  (gr_text 3 (at 143.4485 74.609498) (layer B.SilkS)
+    (effects (font (size 1 1) (thickness 0.2)) (justify mirror))
+  )
+  (gr_text 4 (at 143.4485 76.387498) (layer B.SilkS)
+    (effects (font (size 1 1) (thickness 0.2)) (justify mirror))
+  )
+  (gr_text 1 (at 141.861 74.609498) (layer B.SilkS)
+    (effects (font (size 1 1) (thickness 0.2)) (justify mirror))
+  )
+  (gr_text 2 (at 141.861 76.387498) (layer B.SilkS)
+    (effects (font (size 1 1) (thickness 0.2)) (justify mirror))
   )
   (gr_text V1 (at 113.3495 124.214) (layer B.SilkS)
@@
   (via (at 145.415 118.9609) (size 0.4) (drill 0.3) (layers F.Cu B.Cu) (net 18))
   (via (at 141.605 118.872) (size 0.6) (drill 0.4) (layers F.Cu B.Cu) (net 18))
-  (segment (start 171.218 108.322) (end 171.086 108.19) (width 0.5) (layer B.Cu) (net 19))
-  (segment (start 146.411788 105.71) (end 146.429288 105.7275) (width 0.5) (layer F.Cu) (net 19))
-  (segment (start 145.406 105.71) (end 146.411788 105.71) (width 0.5) (layer F.Cu) (net 19))
-  (segment (start 146.429288 105.7275) (end 148.1455 105.7275) (width 0.5) (layer F.Cu) (net 19))
-  (segment (start 148.1455 105.7275) (end 148.6535 106.2355) (width 0.5) (layer F.Cu) (net 19))
-  (segment (start 148.6535 106.2355) (end 148.6535 112.5855) (width 0.5) (layer F.Cu) (net 19))
-  (segment (start 149.338 113.27) (end 153.306 113.27) (width 0.5) (layer F.Cu) (net 19))
-  (segment (start 148.6535 112.5855) (end 149.338 113.27) (width 0.5) (layer F.Cu) (net 19))
-  (segment (start 161.154 115.582) (end 160.926 115.81) (width 0.5) (layer B.Cu) (net 19))
-  (segment (start 161.154 103.338) (end 160.926 103.11) (width 0.5) (layer B.Cu) (net 19))
-  (segment (start 124.752 63.255) (end 124.761 63.246) (width 0.5) (layer F.Cu) (net 19))
-  (segment (start 123.952 63.255) (end 124.752 63.255) (width 0.5) (layer F.Cu) (net 19))
-  (segment (start 124.761 63.246) (end 126.3015 63.246) (width 0.5) (layer F.Cu) (net 19))
-  (segment (start 127.027 63.9715) (end 127.027 67.8355) (width 0.5) (layer F.Cu) (net 19))
-  (segment (start 126.3015 63.246) (end 127.027 63.9715) (width 0.5) (layer F.Cu) (net 19))
-  (segment (start 127.027 80.518) (end 127.027 84.29) (width 0.5) (layer F.Cu) (net 19))
-  (segment (start 126.274 79.765) (end 127.027 80.518) (width 0.5) (layer F.Cu) (net 19))
-  (segment (start 123.952 79.765) (end 126.274 79.765) (width 0.5) (layer F.Cu) (net 19))
-  (segment (start 155.448 63.255) (end 153.153 63.255) (width 0.5) (layer F.Cu) (net 19))
-  (segment (start 152.427 63.981) (end 152.427 67.8435) (width 0.5) (layer F.Cu) (net 19))
-  (segment (start 153.153 63.255) (end 152.427 63.981) (width 0.5) (layer F.Cu) (net 19))
   (segment (start 154.648 79.765) (end 155.448 79.765) (width 0.5) (layer F.Cu) (net 18))
   (segment (start 154.639 79.756) (end 154.648 79.765) (width 0.5) (layer F.Cu) (net 18))
@@
   (via (at 153.291 117.8005) (size 0.6) (drill 0.4) (layers F.Cu B.Cu) (net 18))
   (via (at 144.147 110.371) (size 0.6) (drill 0.4) (layers F.Cu B.Cu) (net 18))
+  (segment (start 171.218 108.322) (end 171.086 108.19) (width 0.5) (layer B.Cu) (net 19))
+  (segment (start 146.411788 105.71) (end 146.429288 105.7275) (width 0.5) (layer F.Cu) (net 19))
+  (segment (start 145.406 105.71) (end 146.411788 105.71) (width 0.5) (layer F.Cu) (net 19))
+  (segment (start 146.429288 105.7275) (end 148.1455 105.7275) (width 0.5) (layer F.Cu) (net 19))
+  (segment (start 148.1455 105.7275) (end 148.6535 106.2355) (width 0.5) (layer F.Cu) (net 19))
+  (segment (start 148.6535 106.2355) (end 148.6535 112.5855) (width 0.5) (layer F.Cu) (net 19))
+  (segment (start 149.338 113.27) (end 153.306 113.27) (width 0.5) (layer F.Cu) (net 19))
+  (segment (start 148.6535 112.5855) (end 149.338 113.27) (width 0.5) (layer F.Cu) (net 19))
+  (segment (start 161.154 115.582) (end 160.926 115.81) (width 0.5) (layer B.Cu) (net 19))
+  (segment (start 161.154 103.338) (end 160.926 103.11) (width 0.5) (layer B.Cu) (net 19))
+  (segment (start 124.752 63.255) (end 124.761 63.246) (width 0.5) (layer F.Cu) (net 19))
+  (segment (start 123.952 63.255) (end 124.752 63.255) (width 0.5) (layer F.Cu) (net 19))
+  (segment (start 124.761 63.246) (end 126.3015 63.246) (width 0.5) (layer F.Cu) (net 19))
+  (segment (start 127.027 63.9715) (end 127.027 67.8355) (width 0.5) (layer F.Cu) (net 19))
+  (segment (start 126.3015 63.246) (end 127.027 63.9715) (width 0.5) (layer F.Cu) (net 19))
+  (segment (start 127.027 80.518) (end 127.027 84.29) (width 0.5) (layer F.Cu) (net 19))
+  (segment (start 126.274 79.765) (end 127.027 80.518) (width 0.5) (layer F.Cu) (net 19))
+  (segment (start 123.952 79.765) (end 126.274 79.765) (width 0.5) (layer F.Cu) (net 19))
+  (segment (start 155.448 63.255) (end 153.153 63.255) (width 0.5) (layer F.Cu) (net 19))
+  (segment (start 152.427 63.981) (end 152.427 67.8435) (width 0.5) (layer F.Cu) (net 19))
+  (segment (start 153.153 63.255) (end 152.427 63.981) (width 0.5) (layer F.Cu) (net 19))
   (segment (start 165.6 76.075) (end 167.925 76.075) (width 0.5) (layer F.Cu) (net 19))
   (segment (start 168.255 75.745) (end 168.255 74.36) (width 0.5) (layer F.Cu) (net 19))
